File: schematics/Model_CO400.kicad_sch (KiCad schematic)
At the start: 48 parts, among them Q1 PN2222A, SW1 SW_SPST, U1 RE46C107, U2 PIC16F688, U3 MCP6022, U4 TGS-5042

Commit message: Add files via upload
Parts:
- R15: value 600k -> 100K
- R16: value 439k -> 47k
- R17: value 590k -> 470k
Connections:
- net +5V: no longer R17.2
- net GND: no longer U1.9 (REG_{SEL})
- net +3V0 renamed +3V3
- net +3V3: now also R17.2, U1.9 (REG_{SEL})
Other:
- note added: "(5)"
- note added: "(6)"
- note added: "(Amplifier Test 2)"
- note added: "(Sensor Enable/Test1)"
- note added: "**0.298V**"
- note added: "1) Not for production"
- note added: "2) RC0 -> LOW for LED ON & Thermistor Enable"
- note added: "3) RESET (AN3) Causes reset by shorting Vbat"
- note added: "4) TP1 (RA0) has some seral data every 2.5 sec !?!"
- note added: "5) Test1 Modes: 1 HiZ - Normal mode 2 + Vcc ( overrides sensor) read results on AN1 and AN6"
- note added: "6) Test 2 Modes: 1 HiZ - Normal mode ( disables) 2 + Vcc (pulse 0.56 ms) charge C3 for quick reads 3 Analog IN - Reads test voltage int U3a"
- note added: "NOTES:"
- note removed: "(Amplifier Test?)"
- note removed: "(Sensor Enable/Test?)"
- company: 4) TP1 (RA0) has some seral data every 2.5 sec !?! -> (none)
- title: First Alert Model CO400 CO Alarm (ca. 2006) -> First Alert Model CO400 CO Alarm (ca. 2009)
Changed lines of the file:
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@@
 	(paper "A")
 	(title_block
-		(title "First Alert Model CO400 CO Alarm (ca. 2006)")
-		(date "2026-06-04")
-		(rev "A")
-		(company "4) TP1 (RA0) has some seral data every 2.5 sec !?!")
-		(comment 1 "3) RESET (AN3) Causes reset by shorting Vbat ")
-		(comment 2 "2) RC0 -> LOW  for LED ON & Thermistor Enable")
-		(comment 3 "1) Reverse Engineered - there may be errors! ")
-		(comment 4 "NOTES:")
+		(title "First Alert Model CO400 CO Alarm (ca. 2009)")
+		(date "2026-06-10")
+		(rev "B")
+		(comment 2 "B 2026-06-10 Fixed +3V3 Rail and resistor values R15, R16, & R17\"")
+		(comment 3 "A 2026-06-04 Initial Schematic Capture - Caution do not build yet\"! ")
+		(comment 4 "REVISIONS:")
+	)
+	(rectangle
+		(start 232.41 114.3)
+		(end 245.11 116.84)
+		(stroke
+			(width 0)
+			(type default)
+		)
+		(fill
+			(type none)
+		)
 	)
 	(text "(Battery Test?)"
@@
 		)
 	)
+	(text "1) Not for production "
+		(exclude_from_sim no)
+		(at 197.866 20.066 0)
+		(effects
+			(font
+				(size 1.27 1.27)
+			)
+		)
+	)
 	(text "(2)"
 		(exclude_from_sim no)
@@
 		)
 	)
+	(text "(6)"
+		(exclude_from_sim no)
+		(at 149.352 152.908 0)
+		(effects
+			(font
+				(size 1.27 1.27)
+			)
+		)
+	)
 	(text "(Figaro TGS5042)"
 		(exclude_from_sim no)
@@
 		)
 	)
+	(text "NOTES:"
+		(exclude_from_sim no)
+		(at 180.594 16.002 0)
+		(effects
+			(font
+				(size 1.27 1.27)
+			)
+		)
+	)
+	(text "3) RESET (AN3) Causes reset by shorting Vbat "
+		(exclude_from_sim no)
+		(at 186.69 25.908 0)
+		(effects
+			(font
+				(size 1.27 1.27)
+			)
+			(justify left)
+		)
+	)
 	(text "S"
 		(exclude_from_sim no)
@@
 		)
 	)
+	(text "(5)"
+		(exclude_from_sim no)
+		(at 149.86 141.224 0)
+		(effects
+			(font
+				(size 1.27 1.27)
+			)
+		)
+	)
 	(text "(2)"
 		(exclude_from_sim no)
@@
 		)
 	)
+	(text "2) RC0 -> LOW  for LED ON & Thermistor Enable"
+		(exclude_from_sim no)
+		(at 186.69 22.86 0)
+		(effects
+			(font
+				(size 1.27 1.27)
+			)
+			(justify left)
+		)
+	)
 	(text "Alarm & Power "
 		(exclude_from_sim no)
@@
 		)
 	)
-	(text "(Sensor Enable/Test?)"
+	(text "(Sensor Enable/Test1)"
 		(exclude_from_sim no)
-		(at 149.098 133.35 0)
+		(at 148.59 133.604 0)
 		(effects
 			(font
@@
 		)
 	)
+	(text "5) Test1 Modes:\n	1 HiZ - Normal mode  \n	2 + Vcc ( overrides sensor) read results on AN1 and AN6\n"
+		(exclude_from_sim no)
+		(at 186.69 33.02 0)
+		(effects
+			(font
+				(size 1.27 1.27)
+			)
+			(justify left)
+		)
+	)
 	(text "Processor"
 		(exclude_from_sim no)
@@
 		)
 	)
-	(text "(Amplifier Test?) "
+	(text "4) TP1 (RA0) has some seral data every 2.5 sec !?!"
 		(exclude_from_sim no)
-		(at 151.13 154.686 0)
+		(at 186.69 28.448 0)
+		(effects
+			(font
+				(size 1.27 1.27)
+			)
+			(justify left)
+		)
+	)
+	(text "6) Test 2 Modes:\n	1 HiZ - Normal mode ( disables) \n	2 + Vcc (pulse 0.56 ms) charge C3 for quick reads\n	3 Analog IN - Reads test voltage int U3a"
+		(exclude_from_sim no)
+		(at 186.69 40.386 0)
+		(effects
+			(font
+				(size 1.27 1.27)
+			)
+			(justify left)
+		)
+	)
+	(text "**0.298V**"
+		(exclude_from_sim no)
+		(at 238.76 116.078 0)
+		(effects
+			(font
+				(size 1.27 1.27)
+			)
+		)
+	)
+	(text "(Amplifier Test 2) "
+		(exclude_from_sim no)
+		(at 148.082 145.796 0)
 		(effects
 			(font
@@
 	)
 	(junction
+		(at 106.68 63.5)
+		(diameter 0)
+		(color 0 0 0 0)
+	)
+	(junction
 		(at 196.85 104.14)
 		(diameter 0)
@@
 		)
 	)
+	(polyline
+		(pts
+			(xy 219.71 118.11) (xy 222.25 115.57)
+		)
+		(stroke
+			(width 0)
+			(type default)
+		)
+	)
 	(wire
 		(pts
@@
 	(wire
 		(pts
-			(xy 106.68 68.58) (xy 106.68 78.74)
+			(xy 106.68 63.5) (xy 105.41 63.5)
+		)
+		(stroke
+			(width 0)
+			(type default)
+		)
+	)
+	(wire
+		(pts
+			(xy 106.68 63.5) (xy 106.68 68.58)
 		)
 		(stroke
@@
 		)
 	)
+	(polyline
+		(pts
+			(xy 222.25 115.57) (xy 232.41 115.57)
+		)
+		(stroke
+			(width 0)
+			(type default)
+		)
+	)
 	(wire
 		(pts
@@
 	(wire
 		(pts
-			(xy 110.49 63.5) (xy 105.41 63.5)
+			(xy 110.49 63.5) (xy 106.68 63.5)
 		)
 		(stroke
@@
 			)
 		)
-		(property "Value" "439k"
+		(property "Value" "47k"
 			(at 212.344 128.27 90)
 			(effects
@@
 			)
 		)
-		(property "Value" "590k"
+		(property "Value" "470k"
 			(at 226.06 121.92 90)
 			(effects
@@
 			)
 		)
-		(property "Value" "+3V0"
-			(at 113.538 63.5 90)
+		(property "Value" "+3V3"
+			(at 114.046 63.5 0)
 			(effects
 				(font
 					(size 1.27 1.27)
 				)
-				(justify left)
 			)
 		)
@@
 	)
 	(symbol
-		(lib_id "power:GND")
-		(at 106.68 78.74 0)
-		(unit 1)
-		(exclude_from_sim no)
-		(in_bom yes)
-		(on_board yes)
-		(dnp no)
-		(property "Reference" "#PWR011"
-			(at 106.68 85.09 0)
-			(effects
-				(font
-					(size 1.27 1.27)
-				)
-				(hide yes)
-			)
-		)
-		(property "Value" "GND"
-			(at 106.68 83.82 0)
-			(effects
-				(font
-					(size 1.27 1.27)
-				)
-			)
-		)
-		(property "Footprint" ""
-			(at 106.68 78.74 0)
-			(effects
-				(font
-					(size 1.27 1.27)
-				)
-				(hide yes)
-			)
-		)
-		(property "Datasheet" ""
-			(at 106.68 78.74 0)
-			(effects
-				(font
-					(size 1.27 1.27)
-				)
-				(hide yes)
-			)
-		)
-		(property "Description" "Power symbol creates a global label with name \"GND\" , ground"
-			(at 106.68 78.74 0)
-			(effects
-				(font
-					(size 1.27 1.27)
-				)
-				(hide yes)
-			)
-		)
-		(pin "1"
-		)
-		(instances
-			(project "Model_CO400"
-				(path "/409a7a84-5ab7-4d64-8c87-b85c4dc3d66b"
-					(reference "#PWR011")
-					(unit 1)
-				)
-			)
-		)
-	)
-	(symbol
 		(lib_id "Library:R_US")
 		(at 170.18 90.17 90)
@@
 			)
 		)
-		(property "Value" "600k"
+		(property "Value" "100K"
 			(at 162.56 102.8699 0)
 			(effects
@@
 			)
 		)
-		(property "Value" "+3V0"
-			(at 114.3 120.142 90)
+		(property "Value" "+3V3"
+			(at 114.3 119.634 0)
 			(effects
 				(font
 					(size 1.27 1.27)
 				)
-				(justify left)
 			)
 		)
@@
 			)
 		)
-		(property "Value" "+3V0"
-			(at 233.172 52.324 0)
+		(property "Value" "+3V3"
+			(at 236.22 52.324 0)
 			(effects
 				(font
 					(size 1.27 1.27)
 				)
-				(justify left)
 			)
 		)
@@
 			)
 		)
-		(property "Value" "+5V"
+		(property "Value" "+3V3"
 			(at 234.95 125.7299 90)
 			(effects
